File: hydrogen-sensor-pcb.kicad_sch (KiCad schematic)
At the start: 27 parts, among them J1 Conn_01x02_Socket, J2 Conn_01x04_Pin, J3 Conn_01x02_Socket, SW1 SW_Push, U1 STM32F042F6Px, U2 MQ-8, U3 TCAN1043xDxQ1, U4 LD1117S33TR_SOT223, U5 LD1117S50TR_SOT223, Y1 Crystal_GND24

Commit message: Fix border on schematic
Other:
- note added: "Microcontroller"
- note added: "Power supply connector"
- note added: "SWD debug port"
- note added: "TODO: LED (Status PB1, CAN PB8) CAN termination resistor & jumper Check crystal osc values Check viability of used IC (cost, voltage, requriements) Check current MQ-8 sensor current requirements Check if CAN transceiver require more pins connected Annotate document"
- note removed: "STM32"
- note removed: "TODO: LED (Status, CAN) CAN termination resistor & jumper SWD debug port Check crystal osc values"
- moved on the sheet: J2, J3
